File: Hardware_design/uarm_esp32_layout.brd (EAGLE design)
At the start: 16 parts

Commit message: tweaking esp32 layout a bit - 4 in a row
Parts:
- moved E$15 190.5 mm to (304.8, 101.6), turned to 90 degrees
- moved E$14 179.9 mm to (284.5, 141.0), turned to 90 degrees
- moved E$16 172.1 mm to (287.0, 120.7), turned to 180 degrees
- moved E$10 85.2 mm to (-17.8, 120.7)
- moved E$3 85.2 mm to (-172.7, 141.0)
- moved E$6 85.2 mm to (-152.4, 101.6)
- moved E$7 85.2 mm to (-170.2, 120.7)
- moved E$8 85.2 mm to (-20.3, 141.0)
- moved E$9 85.2 mm to (0.00, 101.6)
- moved E$11 85.2 mm to (132.1, 141.0)
- moved E$12 85.2 mm to (152.4, 101.6)
- moved E$13 85.2 mm to (134.6, 120.7)
- moved E$17 68.4 mm to (-166.4, 55.9)
- moved E$18 68.4 mm to (-127.0, 76.2)
- moved E$19 68.4 mm to (-146.1, 58.4)
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Changed lines of the file:
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@@
 </autorouter>
 <elements>
-<element name="E$1" library="sandbox" package="UARM" value="" x="0" y="0" rot="R90"/>
-<element name="E$3" library="uarm_alignment_base" package="CARTRIDGE_ESP32" value="" x="-96.52" y="179.07" rot="R90"/>
-<element name="E$6" library="SparkFun-Hardware" package="ACTOBOTICS_CHANNEL_6&quot;" value="" x="-76.2" y="139.7" rot="R90"/>
-<element name="E$7" library="uarm_alignment_base" package="UARM_ALIGNMENT_BASE" value="" x="-93.98" y="158.75" rot="R180"/>
-<element name="E$8" library="uarm_alignment_base" package="CARTRIDGE_ESP32" value="" x="55.88" y="179.07" rot="R90"/>
-<element name="E$9" library="SparkFun-Hardware" package="ACTOBOTICS_CHANNEL_6&quot;" value="" x="76.2" y="139.7" rot="R90"/>
-<element name="E$10" library="uarm_alignment_base" package="UARM_ALIGNMENT_BASE" value="" x="58.42" y="158.75" rot="R180"/>
-<element name="E$11" library="uarm_alignment_base" package="CARTRIDGE_ESP32" value="" x="208.28" y="179.07" rot="R90"/>
-<element name="E$12" library="SparkFun-Hardware" package="ACTOBOTICS_CHANNEL_6&quot;" value="" x="228.6" y="139.7" rot="R90"/>
-<element name="E$13" library="uarm_alignment_base" package="UARM_ALIGNMENT_BASE" value="" x="210.82" y="158.75" rot="R180"/>
-<element name="E$14" library="uarm_alignment_base" package="CARTRIDGE_ESP32" value="" x="229.87" y="-30.48"/>
-<element name="E$15" library="SparkFun-Hardware" package="ACTOBOTICS_CHANNEL_6&quot;" value="" x="190.5" y="-50.8"/>
-<element name="E$16" library="uarm_alignment_base" package="UARM_ALIGNMENT_BASE" value="" x="209.55" y="-33.02" rot="R90"/>
-<element name="E$17" library="uarm_alignment_base" package="CARTRIDGE_ESP32" value="" x="-229.87" y="81.28" rot="R180"/>
-<element name="E$18" library="SparkFun-Hardware" package="ACTOBOTICS_CHANNEL_6&quot;" value="" x="-190.5" y="101.6" rot="R180"/>
-<element name="E$19" library="uarm_alignment_base" package="UARM_ALIGNMENT_BASE" value="" x="-209.55" y="83.82" rot="R270"/>
+<element name="E$1" library="sandbox" package="UARM" value="" x="0" y="0" rot="R100"/>
+<element name="E$3" library="uarm_alignment_base" package="CARTRIDGE_ESP32" value="" x="-172.72" y="140.97" rot="R90"/>
+<element name="E$6" library="SparkFun-Hardware" package="ACTOBOTICS_CHANNEL_6&quot;" value="" x="-152.4" y="101.6" rot="R90"/>
+<element name="E$7" library="uarm_alignment_base" package="UARM_ALIGNMENT_BASE" value="" x="-170.18" y="120.65" rot="R180"/>
+<element name="E$8" library="uarm_alignment_base" package="CARTRIDGE_ESP32" value="" x="-20.32" y="140.97" rot="R90"/>
+<element name="E$9" library="SparkFun-Hardware" package="ACTOBOTICS_CHANNEL_6&quot;" value="" x="0" y="101.6" rot="R90"/>
+<element name="E$10" library="uarm_alignment_base" package="UARM_ALIGNMENT_BASE" value="" x="-17.78" y="120.65" rot="R180"/>
+<element name="E$11" library="uarm_alignment_base" package="CARTRIDGE_ESP32" value="" x="132.08" y="140.97" rot="R90"/>
+<element name="E$12" library="SparkFun-Hardware" package="ACTOBOTICS_CHANNEL_6&quot;" value="" x="152.4" y="101.6" rot="R90"/>
+<element name="E$13" library="uarm_alignment_base" package="UARM_ALIGNMENT_BASE" value="" x="134.62" y="120.65" rot="R180"/>
+<element name="E$14" library="uarm_alignment_base" package="CARTRIDGE_ESP32" value="" x="284.48" y="140.97" rot="R90"/>
+<element name="E$15" library="SparkFun-Hardware" package="ACTOBOTICS_CHANNEL_6&quot;" value="" x="304.8" y="101.6" rot="R90"/>
+<element name="E$16" library="uarm_alignment_base" package="UARM_ALIGNMENT_BASE" value="" x="287.02" y="120.65" rot="R180"/>
+<element name="E$17" library="uarm_alignment_base" package="CARTRIDGE_ESP32" value="" x="-166.37" y="55.88" rot="R180"/>
+<element name="E$18" library="SparkFun-Hardware" package="ACTOBOTICS_CHANNEL_6&quot;" value="" x="-127" y="76.2" rot="R180"/>
+<element name="E$19" library="uarm_alignment_base" package="UARM_ALIGNMENT_BASE" value="" x="-146.05" y="58.42" rot="R270"/>
 </elements>
 <signals>

Commit message: tweaking hardware layout
Parts:
- added E$2, E$20, E$21, E$22, E$23, E$4, E$5: (no value), SparkFun-Hardware:ACTOBOTICS_CHANNEL_SINGLE_DRILL_REF
- added E$24: (no value), uarm_alignment_base:ACTOBOTICS_BEAM_4.62_INCH
- moved E$6 256.0 mm to (-406.4, 69.8)
Changed lines of the file:
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@@
 <setting verticaltext="up"/>
 </settings>
-<grid distance="0.5" unitdist="inch" unit="inch" style="lines" multiple="1" display="yes" altdistance="0.005" altunitdist="inch" altunit="inch"/>
+<grid distance="0.25" unitdist="inch" unit="inch" style="lines" multiple="1" display="yes" altdistance="0.005" altunitdist="inch" altunit="inch"/>
 <layers>
 <layer number="1" name="Top" color="4" fill="1" visible="yes" active="yes"/>
@@
 <element name="E$1" library="sandbox" package="UARM" value="" x="0" y="0" rot="R100"/>
 <element name="E$3" library="uarm_alignment_base" package="CARTRIDGE_ESP32" value="" x="-172.72" y="140.97" rot="R90"/>
-<element name="E$6" library="SparkFun-Hardware" package="ACTOBOTICS_CHANNEL_6&quot;" value="" x="-152.4" y="101.6" rot="R90"/>
+<element name="E$6" library="SparkFun-Hardware" package="ACTOBOTICS_CHANNEL_6&quot;" value="" x="-406.4" y="69.85" rot="R90"/>
 <element name="E$7" library="uarm_alignment_base" package="UARM_ALIGNMENT_BASE" value="" x="-170.18" y="120.65" rot="R180"/>
 <element name="E$8" library="uarm_alignment_base" package="CARTRIDGE_ESP32" value="" x="-20.32" y="140.97" rot="R90"/>
@@
 <element name="E$18" library="SparkFun-Hardware" package="ACTOBOTICS_CHANNEL_6&quot;" value="" x="-127" y="76.2" rot="R180"/>
 <element name="E$19" library="uarm_alignment_base" package="UARM_ALIGNMENT_BASE" value="" x="-146.05" y="58.42" rot="R270"/>
+<element name="E$2" library="SparkFun-Hardware" package="ACTOBOTICS_CHANNEL_SINGLE_DRILL_REF" value="" x="-482.6" y="69.85" rot="R90"/>
+<element name="E$4" library="SparkFun-Hardware" package="ACTOBOTICS_CHANNEL_SINGLE_DRILL_REF" value="" x="-501.65" y="69.85" rot="R90"/>
+<element name="E$5" library="SparkFun-Hardware" package="ACTOBOTICS_CHANNEL_SINGLE_DRILL_REF" value="" x="-520.7" y="69.85" rot="R90"/>
+<element name="E$20" library="SparkFun-Hardware" package="ACTOBOTICS_CHANNEL_SINGLE_DRILL_REF" value="" x="-463.55" y="69.85" rot="R90"/>
+<element name="E$21" library="SparkFun-Hardware" package="ACTOBOTICS_CHANNEL_SINGLE_DRILL_REF" value="" x="-444.5" y="69.85" rot="R90"/>
+<element name="E$22" library="SparkFun-Hardware" package="ACTOBOTICS_CHANNEL_SINGLE_DRILL_REF" value="" x="-425.45" y="69.85" rot="R90"/>
+<element name="E$23" library="SparkFun-Hardware" package="ACTOBOTICS_CHANNEL_SINGLE_DRILL_REF" value="" x="-406.4" y="69.85" rot="R90"/>
+<element name="E$24" library="uarm_alignment_base" package="ACTOBOTICS_BEAM_4.62_INCH" value="" x="-539.75" y="120.65"/>
 </elements>
 <signals>
@@
 </board>
 </drawing>
+<compatibility>
+<note version="6.3" minversion="6.2.2" severity="warning">
+Since Version 6.2.2 text objects can contain more than one line,
+which will not be processed correctly with this version.
+</note>
+</compatibility>
 </eagle>

Commit message: more hardware layout ideas
added 18x24 laser cutter maz package for reference. Thinking that I may
cut the "base" of this table top with the lazer cutter, so I don't have
to manually measure and drill all these mounting holes.
Parts:
- removed E$24: (no value), uarm_alignment_base:ACTOBOTICS_BEAM_4.62_INCH
- added E$25: (no value), uarm_alignment_base:LASER_CUTTER_MAX_SIZE
- moved E$4 808.5 mm to (304.8, 127.0)
- moved E$20 637.6 mm to (171.4, 127.0)
- moved E$5 542.8 mm to (19.1, 127.0)
- moved E$21 318.1 mm to (-127.0, 88.9), turned to 180 degrees
- moved E$22 313.3 mm to (-127.0, -25.4), turned to 180 degrees
- moved E$23 279.0 mm to (-133.3, 127.0)
- moved E$6 260.3 mm to (-152.4, 127.0)
- moved E$2 223.3 mm to (-266.7, 127.0)
- moved E$10 25.4 mm to (-17.8, 146.1)
- moved E$11 25.4 mm to (132.1, 166.4)
- moved E$12 25.4 mm to (152.4, 127.0)
- moved E$13 25.4 mm to (134.6, 146.1)
- moved E$14 25.4 mm to (284.5, 166.4)
- moved E$15 25.4 mm to (304.8, 127.0)
- moved E$16 25.4 mm to (287.0, 146.1)
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Changed lines of the file:
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@@
 <setting verticaltext="up"/>
 </settings>
-<grid distance="0.25" unitdist="inch" unit="inch" style="lines" multiple="1" display="yes" altdistance="0.005" altunitdist="inch" altunit="inch"/>
+<grid distance="0.5" unitdist="inch" unit="inch" style="lines" multiple="1" display="yes" altdistance="0.25" altunitdist="inch" altunit="inch"/>
 <layers>
 <layer number="1" name="Top" color="4" fill="1" visible="yes" active="yes"/>
@@
 <elements>
 <element name="E$1" library="sandbox" package="UARM" value="" x="0" y="0" rot="R100"/>
-<element name="E$3" library="uarm_alignment_base" package="CARTRIDGE_ESP32" value="" x="-172.72" y="140.97" rot="R90"/>
-<element name="E$6" library="SparkFun-Hardware" package="ACTOBOTICS_CHANNEL_6&quot;" value="" x="-406.4" y="69.85" rot="R90"/>
-<element name="E$7" library="uarm_alignment_base" package="UARM_ALIGNMENT_BASE" value="" x="-170.18" y="120.65" rot="R180"/>
-<element name="E$8" library="uarm_alignment_base" package="CARTRIDGE_ESP32" value="" x="-20.32" y="140.97" rot="R90"/>
-<element name="E$9" library="SparkFun-Hardware" package="ACTOBOTICS_CHANNEL_6&quot;" value="" x="0" y="101.6" rot="R90"/>
-<element name="E$10" library="uarm_alignment_base" package="UARM_ALIGNMENT_BASE" value="" x="-17.78" y="120.65" rot="R180"/>
-<element name="E$11" library="uarm_alignment_base" package="CARTRIDGE_ESP32" value="" x="132.08" y="140.97" rot="R90"/>
-<element name="E$12" library="SparkFun-Hardware" package="ACTOBOTICS_CHANNEL_6&quot;" value="" x="152.4" y="101.6" rot="R90"/>
-<element name="E$13" library="uarm_alignment_base" package="UARM_ALIGNMENT_BASE" value="" x="134.62" y="120.65" rot="R180"/>
-<element name="E$14" library="uarm_alignment_base" package="CARTRIDGE_ESP32" value="" x="284.48" y="140.97" rot="R90"/>
-<element name="E$15" library="SparkFun-Hardware" package="ACTOBOTICS_CHANNEL_6&quot;" value="" x="304.8" y="101.6" rot="R90"/>
-<element name="E$16" library="uarm_alignment_base" package="UARM_ALIGNMENT_BASE" value="" x="287.02" y="120.65" rot="R180"/>
-<element name="E$17" library="uarm_alignment_base" package="CARTRIDGE_ESP32" value="" x="-166.37" y="55.88" rot="R180"/>
-<element name="E$18" library="SparkFun-Hardware" package="ACTOBOTICS_CHANNEL_6&quot;" value="" x="-127" y="76.2" rot="R180"/>
-<element name="E$19" library="uarm_alignment_base" package="UARM_ALIGNMENT_BASE" value="" x="-146.05" y="58.42" rot="R270"/>
-<element name="E$2" library="SparkFun-Hardware" package="ACTOBOTICS_CHANNEL_SINGLE_DRILL_REF" value="" x="-482.6" y="69.85" rot="R90"/>
-<element name="E$4" library="SparkFun-Hardware" package="ACTOBOTICS_CHANNEL_SINGLE_DRILL_REF" value="" x="-501.65" y="69.85" rot="R90"/>
-<element name="E$5" library="SparkFun-Hardware" package="ACTOBOTICS_CHANNEL_SINGLE_DRILL_REF" value="" x="-520.7" y="69.85" rot="R90"/>
-<element name="E$20" library="SparkFun-Hardware" package="ACTOBOTICS_CHANNEL_SINGLE_DRILL_REF" value="" x="-463.55" y="69.85" rot="R90"/>
-<element name="E$21" library="SparkFun-Hardware" package="ACTOBOTICS_CHANNEL_SINGLE_DRILL_REF" value="" x="-444.5" y="69.85" rot="R90"/>
-<element name="E$22" library="SparkFun-Hardware" package="ACTOBOTICS_CHANNEL_SINGLE_DRILL_REF" value="" x="-425.45" y="69.85" rot="R90"/>
-<element name="E$23" library="SparkFun-Hardware" package="ACTOBOTICS_CHANNEL_SINGLE_DRILL_REF" value="" x="-406.4" y="69.85" rot="R90"/>
-<element name="E$24" library="uarm_alignment_base" package="ACTOBOTICS_BEAM_4.62_INCH" value="" x="-539.75" y="120.65"/>
+<element name="E$3" library="uarm_alignment_base" package="CARTRIDGE_ESP32" value="" x="-172.72" y="166.37" rot="R90"/>
+<element name="E$6" library="SparkFun-Hardware" package="ACTOBOTICS_CHANNEL_6&quot;" value="" x="-152.4" y="127" rot="R90"/>
+<element name="E$7" library="uarm_alignment_base" package="UARM_ALIGNMENT_BASE" value="" x="-170.18" y="146.05" rot="R180"/>
+<element name="E$8" library="uarm_alignment_base" package="CARTRIDGE_ESP32" value="" x="-20.32" y="166.37" rot="R90"/>
+<element name="E$9" library="SparkFun-Hardware" package="ACTOBOTICS_CHANNEL_6&quot;" value="" x="0" y="127" rot="R90"/>
+<element name="E$10" library="uarm_alignment_base" package="UARM_ALIGNMENT_BASE" value="" x="-17.78" y="146.05" rot="R180"/>
+<element name="E$11" library="uarm_alignment_base" package="CARTRIDGE_ESP32" value="" x="132.08" y="166.37" rot="R90"/>
+<element name="E$12" library="SparkFun-Hardware" package="ACTOBOTICS_CHANNEL_6&quot;" value="" x="152.4" y="127" rot="R90"/>
+<element name="E$13" library="uarm_alignment_base" package="UARM_ALIGNMENT_BASE" value="" x="134.62" y="146.05" rot="R180"/>
+<element name="E$14" library="uarm_alignment_base" package="CARTRIDGE_ESP32" value="" x="284.48" y="166.37" rot="R90"/>
+<element name="E$15" library="SparkFun-Hardware" package="ACTOBOTICS_CHANNEL_6&quot;" value="" x="304.8" y="127" rot="R90"/>
+<element name="E$16" library="uarm_alignment_base" package="UARM_ALIGNMENT_BASE" value="" x="287.02" y="146.05" rot="R180"/>
+<element name="E$17" library="uarm_alignment_base" package="CARTRIDGE_ESP32" value="" x="-166.37" y="68.58" rot="R180"/>
+<element name="E$18" library="SparkFun-Hardware" package="ACTOBOTICS_CHANNEL_6&quot;" value="" x="-127" y="88.9" rot="R180"/>
+<element name="E$19" library="uarm_alignment_base" package="UARM_ALIGNMENT_BASE" value="" x="-146.05" y="71.12" rot="R270"/>
+<element name="E$2" library="SparkFun-Hardware" package="ACTOBOTICS_CHANNEL_SINGLE_DRILL_REF" value="" x="-266.7" y="127" rot="R90"/>
+<element name="E$23" library="SparkFun-Hardware" package="ACTOBOTICS_CHANNEL_SINGLE_DRILL_REF" value="" x="-133.35" y="127" rot="R90"/>
+<element name="E$25" library="uarm_alignment_base" package="LASER_CUTTER_MAX_SIZE" value="" x="-304.8" y="-292.1"/>
+<element name="E$4" library="SparkFun-Hardware" package="ACTOBOTICS_CHANNEL_SINGLE_DRILL_REF" value="" x="304.8" y="127" rot="R90"/>
+<element name="E$5" library="SparkFun-Hardware" package="ACTOBOTICS_CHANNEL_SINGLE_DRILL_REF" value="" x="19.05" y="127" rot="R90"/>
+<element name="E$20" library="SparkFun-Hardware" package="ACTOBOTICS_CHANNEL_SINGLE_DRILL_REF" value="" x="171.45" y="127" rot="R90"/>
+<element name="E$21" library="SparkFun-Hardware" package="ACTOBOTICS_CHANNEL_SINGLE_DRILL_REF" value="" x="-127" y="88.9" rot="R180"/>
+<element name="E$22" library="SparkFun-Hardware" package="ACTOBOTICS_CHANNEL_SINGLE_DRILL_REF" value="" x="-127" y="-25.4" rot="R180"/>
 </elements>
 <signals>
