File: Hardware_design/Cartridge_belt.brd (EAGLE design)
At the start: 1 part

Commit message: Mote work on belt wall design
Parts:
- added E$2, E$3, E$4, E$5: (no value), SparkFun-Hardware:ACTOBOTICS_CHANNEL_SINGLE_DRILL_REF

Commit message: More belt fine tuning
created packages for some of the gears/rods
Parts:
- added E$10, E$6, E$9: (no value), uarm_alignment_base:TUBE_&_BEARING_1/2"
- added E$11, E$12: (no value), SparkFun-Hardware:ACTOBOTICS_CHANNEL_SINGLE_DRILL_REF
- added E$7, E$8: (no value), uarm_alignment_base:GEAR_84T
- moved E$1 38.1 mm to (25.4, 673.1)
- moved E$2 38.1 mm to (0.00, 571.5)
- moved E$3 38.1 mm to (114.3, 571.5)
Changed lines of the file:
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@@
 <setting verticaltext="up"/>
 </settings>
-<grid distance="0.5" unitdist="inch" unit="inch" style="lines" multiple="1" display="yes" altdistance="0.1" altunitdist="inch" altunit="inch"/>
+<grid distance="0.5" unitdist="inch" unit="inch" style="lines" multiple="1" display="yes" altdistance="0.005" altunitdist="inch" altunit="inch"/>
 <layers>
 <layer number="1" name="Top" color="4" fill="1" visible="yes" active="yes"/>
@@
 <board>
 <plain>
-<wire x1="0" y1="0" x2="0" y2="647.7" width="0.254" layer="49"/>
-<wire x1="0" y1="647.7" x2="152.4" y2="647.7" width="0.254" layer="49"/>
-<wire x1="152.4" y1="647.7" x2="152.4" y2="0" width="0.254" layer="49"/>
+<wire x1="0" y1="0" x2="0" y2="609.6" width="0.254" layer="49"/>
+<wire x1="0" y1="609.6" x2="152.4" y2="609.6" width="0.254" layer="49"/>
+<wire x1="152.4" y1="609.6" x2="152.4" y2="0" width="0.254" layer="49"/>
 <wire x1="152.4" y1="0" x2="0" y2="0" width="0.254" layer="49"/>
-<circle x="38.1" y="596.9" radius="6.35" width="0.254" layer="51"/>
-<wire x1="50.8" y1="584.2" x2="50.8" y2="114.3" width="6.35" layer="51"/>
-<wire x1="101.6" y1="584.2" x2="101.6" y2="114.3" width="6.35" layer="51"/>
-<circle x="57.15" y="16.256" radius="7.184203125" width="0.254" layer="49"/>
-<wire x1="85.09" y1="25.4" x2="85.09" y2="7.874" width="0.254" layer="49"/>
-<wire x1="85.09" y1="7.874" x2="84.836" y2="7.62" width="0.254" layer="49" curve="-90"/>
-<wire x1="84.836" y1="7.62" x2="46.99" y2="7.62" width="0.254" layer="49"/>
-<wire x1="46.99" y1="7.62" x2="46.99" y2="25.146" width="0.254" layer="49"/>
-<wire x1="46.99" y1="25.146" x2="47.244" y2="25.4" width="0.254" layer="49" curve="-90"/>
-<wire x1="47.244" y1="25.4" x2="85.09" y2="25.4" width="0.254" layer="49"/>
-<circle x="107.696" y="55.626" radius="34.036" width="0.254" layer="49"/>
-<circle x="39.878" y="55.118" radius="34.036" width="0.254" layer="49"/>
-<circle x="107.696" y="55.626" radius="5.08" width="0.254" layer="51"/>
-<circle x="39.878" y="55.118" radius="5.08" width="0.254" layer="51"/>
-<text x="36.83" y="85.09" size="1.778" layer="49" font="vector" ratio="15">84T</text>
-<circle x="24.638" y="40.386" radius="6.35" width="0.254" layer="51"/>
-<circle x="57.15" y="42.418" radius="6.35" width="0.254" layer="51"/>
-<wire x1="34.798" y1="57.912" x2="34.29" y2="52.324" width="0.6096" layer="21" curve="43.759612"/>
-<wire x1="30.988" y1="597.154" x2="38.1" y2="604.52" width="0.6096" layer="21" curve="-83.121022"/>
-<wire x1="38.1" y1="604.52" x2="43.434" y2="601.98" width="0.6096" layer="21" curve="-59.815707"/>
-<wire x1="43.434" y1="601.98" x2="53.594" y2="587.502" width="0.6096" layer="21" curve="0.861296"/>
-<wire x1="53.594" y1="587.502" x2="54.61" y2="583.438" width="0.6096" layer="21" curve="-42.907665"/>
-<wire x1="54.61" y1="583.438" x2="54.61" y2="113.03" width="0.6096" layer="21"/>
-<dimension x1="139.7" y1="622.3" x2="139.7" y2="711.2" x3="203.2" y3="666.75" textsize="1.778" textratio="15" layer="21" unit="inch"/>
-<wire x1="54.61" y1="113.03" x2="34.29" y2="56.769" width="0.6096" layer="21"/>
-<wire x1="34.29" y1="56.769" x2="40.386" y2="49.403" width="0.6096" layer="21" curve="118.93816"/>
-<wire x1="40.64" y1="49.53" x2="57.15" y2="49.53" width="0.6096" layer="21"/>
-<wire x1="57.15" y1="49.53" x2="64.77" y2="41.91" width="0.6096" layer="21" curve="-90"/>
-<wire x1="64.77" y1="41.91" x2="58.42" y2="35.56" width="0.6096" layer="21" curve="-90"/>
-<wire x1="58.42" y1="35.56" x2="24.765" y2="33.528" width="0.6096" layer="21"/>
-<wire x1="24.765" y1="33.528" x2="17.78" y2="41.148" width="0.6096" layer="21" curve="-101.889589"/>
-<wire x1="17.78" y1="41.148" x2="30.988" y2="596.9" width="0.6096" layer="21"/>
+<wire x1="50.8" y1="546.1" x2="50.8" y2="101.6" width="6.35" layer="51"/>
+<wire x1="101.6" y1="546.1" x2="101.6" y2="101.6" width="6.35" layer="51"/>
+<circle x="48.910396875" y="19.00886875" radius="7.184203125" width="0.254" layer="49"/>
+<wire x1="78.013765625" y1="23.162221875" x2="74.970409375" y2="5.90248125" width="0.254" layer="49"/>
+<wire x1="74.970409375" y1="5.90248125" x2="74.676159375" y2="5.696446875" width="0.254" layer="49" curve="-90"/>
+<wire x1="74.676159375" y1="5.696446875" x2="37.405125" y2="12.268334375" width="0.254" layer="49"/>
+<wire x1="37.405125" y1="12.268334375" x2="40.448484375" y2="29.528075" width="0.254" layer="49"/>
+<wire x1="40.448484375" y1="29.528075" x2="40.74273125" y2="29.7341125" width="0.254" layer="49" curve="-90"/>
+<wire x1="40.74273125" y1="29.7341125" x2="78.013765625" y2="23.162221875" width="0.254" layer="49"/>
+<text x="36.83" y="72.39" size="1.778" layer="49" font="vector" ratio="15">84T</text>
+<wire x1="31.242" y1="559.054" x2="37.338" y2="565.531" width="0.6096" layer="21" curve="-83.121022"/>
+<wire x1="37.338" y1="565.531" x2="42.799" y2="563.626" width="0.6096" layer="21" curve="-59.815707"/>
+<wire x1="42.799" y1="563.626" x2="53.594" y2="548.513" width="0.6096" layer="21" curve="0.861296"/>
+<wire x1="53.594" y1="548.513" x2="54.61" y2="545.338" width="0.6096" layer="21" curve="-42.907665"/>
+<wire x1="54.61" y1="545.338" x2="54.61" y2="100.33" width="0.6096" layer="21"/>
+<dimension x1="139.7" y1="584.2" x2="139.7" y2="673.1" x3="203.2" y3="628.65" textsize="1.778" textratio="15" layer="21" unit="inch"/>
+<wire x1="54.61" y1="100.33" x2="34.29" y2="64.008" width="0.6096" layer="21"/>
+<wire x1="34.29" y1="64.008" x2="44.069" y2="51.308" width="0.6096" layer="21" curve="118.93816"/>
+<wire x1="44.069" y1="51.308" x2="59.182" y2="51.181" width="0.6096" layer="21"/>
+<wire x1="59.182" y1="51.181" x2="65.532" y2="43.561" width="0.6096" layer="21" curve="-90"/>
+<wire x1="65.532" y1="43.561" x2="58.928" y2="37.338" width="0.6096" layer="21" curve="-90"/>
+<wire x1="58.928" y1="37.338" x2="21.844" y2="37.465" width="0.6096" layer="21"/>
+<wire x1="21.844" y1="37.465" x2="15.113" y2="45.212" width="0.6096" layer="21" curve="-101.889589"/>
+<wire x1="15.113" y1="45.212" x2="31.242" y2="559.054" width="0.6096" layer="21"/>
+<wire x1="76.2" y1="-50.8" x2="76.2" y2="723.9" width="0.254" layer="49" style="longdash"/>
 </plain>
 <attributes>
@@
 </autorouter>
 <elements>
-<element name="E$1" library="uarm_alignment_base" package="CARTRIDGE_ESP32" value="" x="25.4" y="711.2" rot="R270"/>
-<element name="E$2" library="SparkFun-Hardware" package="ACTOBOTICS_CHANNEL_SINGLE_DRILL_REF" value="" x="0" y="609.6"/>
-<element name="E$3" library="SparkFun-Hardware" package="ACTOBOTICS_CHANNEL_SINGLE_DRILL_REF" value="" x="114.3" y="609.6"/>
+<element name="E$1" library="uarm_alignment_base" package="CARTRIDGE_ESP32" value="" x="25.4" y="673.1" rot="R270"/>
+<element name="E$2" library="SparkFun-Hardware" package="ACTOBOTICS_CHANNEL_SINGLE_DRILL_REF" value="" x="0" y="571.5"/>
+<element name="E$3" library="SparkFun-Hardware" package="ACTOBOTICS_CHANNEL_SINGLE_DRILL_REF" value="" x="114.3" y="571.5"/>
 <element name="E$4" library="SparkFun-Hardware" package="ACTOBOTICS_CHANNEL_SINGLE_DRILL_REF" value="" x="0" y="0"/>
 <element name="E$5" library="SparkFun-Hardware" package="ACTOBOTICS_CHANNEL_SINGLE_DRILL_REF" value="" x="114.3" y="0"/>
+<element name="E$6" library="uarm_alignment_base" package="TUBE_&amp;_BEARING_1/2&quot;" value="" x="38.1" y="558.8"/>
+<element name="E$7" library="uarm_alignment_base" package="GEAR_84T" value="" x="109.601" y="60.325"/>
+<element name="E$8" library="uarm_alignment_base" package="GEAR_84T" value="" x="42.799" y="60.325"/>
+<element name="E$9" library="uarm_alignment_base" package="TUBE_&amp;_BEARING_1/2&quot;" value="" x="58.547" y="44.196"/>
+<element name="E$10" library="uarm_alignment_base" package="TUBE_&amp;_BEARING_1/2&quot;" value="" x="21.844" y="44.069"/>
+<element name="E$11" library="SparkFun-Hardware" package="ACTOBOTICS_CHANNEL_SINGLE_DRILL_REF" value="" x="0" y="508"/>
+<element name="E$12" library="SparkFun-Hardware" package="ACTOBOTICS_CHANNEL_SINGLE_DRILL_REF" value="" x="114.3" y="508"/>
 </elements>
 <signals>

Commit message: more belt perfection
Scooted top point up to better match pick hieght of current arm setup.

Adjusted width of belt rack walls (made them tighter to more accurately
fit the esp32 board).

Added in some belt widt lines that are more precise on a high layer
number.

total belt length is now 46.1 inches. Ordered the 46" belt, hope it
won't be too tight, could always adjust the roll tubes to adjust
tightness.

still need to plan for the switches.
Parts:
- moved E$1 90.5 mm to (21.0, 582.7)
- moved E$11 25.4 mm to (0.00, 533.4)
- moved E$12 25.4 mm to (114.3, 533.4)
- moved E$6 22.1 mm to (56.1, 571.6)
Changed lines of the file:
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@@
 <setting verticaltext="up"/>
 </settings>
-<grid distance="0.5" unitdist="inch" unit="inch" style="lines" multiple="1" display="yes" altdistance="0.005" altunitdist="inch" altunit="inch"/>
+<grid distance="0.5" unitdist="inch" unit="inch" style="lines" multiple="1" display="yes" altdistance="0.05" altunitdist="inch" altunit="inch"/>
 <layers>
 <layer number="1" name="Top" color="4" fill="1" visible="yes" active="yes"/>
@@
 <layer number="45" name="Holes" color="7" fill="1" visible="yes" active="yes"/>
 <layer number="46" name="Milling" color="3" fill="1" visible="no" active="yes"/>
-<layer number="47" name="Measures" color="7" fill="1" visible="no" active="yes"/>
+<layer number="47" name="Measures" color="7" fill="1" visible="yes" active="yes"/>
 <layer number="48" name="Document" color="7" fill="1" visible="no" active="yes"/>
 <layer number="49" name="Reference" color="13" fill="1" visible="yes" active="yes"/>
@@
 <layer number="106" name="bPlate" color="7" fill="1" visible="no" active="yes"/>
 <layer number="107" name="Crop" color="7" fill="1" visible="no" active="yes"/>
-<layer number="108" name="tplace-old" color="10" fill="1" visible="no" active="yes"/>
+<layer number="108" name="tplace-old" color="10" fill="1" visible="yes" active="yes"/>
 <layer number="109" name="ref-old" color="11" fill="1" visible="no" active="yes"/>
 <layer number="110" name="fp0" color="7" fill="1" visible="no" active="yes"/>
@@
 <plain>
 <wire x1="0" y1="0" x2="0" y2="609.6" width="0.254" layer="49"/>
-<wire x1="0" y1="609.6" x2="152.4" y2="609.6" width="0.254" layer="49"/>
+<wire x1="0" y1="609.6" x2="44.45" y2="609.6" width="0.254" layer="49"/>
+<wire x1="44.45" y1="609.6" x2="69.85" y2="584.2" width="0.254" layer="49"/>
+<wire x1="69.85" y1="584.2" x2="82.55" y2="584.2" width="0.254" layer="49"/>
+<wire x1="82.55" y1="584.2" x2="107.95" y2="609.6" width="0.254" layer="49"/>
+<wire x1="107.95" y1="609.6" x2="152.4" y2="609.6" width="0.254" layer="49"/>
 <wire x1="152.4" y1="609.6" x2="152.4" y2="0" width="0.254" layer="49"/>
 <wire x1="152.4" y1="0" x2="0" y2="0" width="0.254" layer="49"/>
-<wire x1="50.8" y1="546.1" x2="50.8" y2="101.6" width="6.35" layer="51"/>
-<wire x1="101.6" y1="546.1" x2="101.6" y2="101.6" width="6.35" layer="51"/>
+<wire x1="59.309" y1="571.5" x2="59.309" y2="99.06" width="6.35" layer="51"/>
+<wire x1="94.361" y1="571.5" x2="94.361" y2="99.06" width="6.35" layer="51"/>
 <circle x="48.910396875" y="19.00886875" radius="7.184203125" width="0.254" layer="49"/>
 <wire x1="78.013765625" y1="23.162221875" x2="74.970409375" y2="5.90248125" width="0.254" layer="49"/>
@@
 <wire x1="40.74273125" y1="29.7341125" x2="78.013765625" y2="23.162221875" width="0.254" layer="49"/>
 <text x="36.83" y="72.39" size="1.778" layer="49" font="vector" ratio="15">84T</text>
-<wire x1="31.242" y1="559.054" x2="37.338" y2="565.531" width="0.6096" layer="21" curve="-83.121022"/>
-<wire x1="37.338" y1="565.531" x2="42.799" y2="563.626" width="0.6096" layer="21" curve="-59.815707"/>
-<wire x1="42.799" y1="563.626" x2="53.594" y2="548.513" width="0.6096" layer="21" curve="0.861296"/>
-<wire x1="53.594" y1="548.513" x2="54.61" y2="545.338" width="0.6096" layer="21" curve="-42.907665"/>
-<wire x1="54.61" y1="545.338" x2="54.61" y2="100.33" width="0.6096" layer="21"/>
-<dimension x1="139.7" y1="584.2" x2="139.7" y2="673.1" x3="203.2" y3="628.65" textsize="1.778" textratio="15" layer="21" unit="inch"/>
-<wire x1="54.61" y1="100.33" x2="34.29" y2="64.008" width="0.6096" layer="21"/>
+<wire x1="49.276" y1="571.881" x2="55.372" y2="578.358" width="0.6096" layer="21" curve="-83.121022"/>
+<wire x1="55.372" y1="578.358" x2="61.468" y2="576.072" width="0.6096" layer="21" curve="-59.815707"/>
+<wire x1="61.468" y1="576.072" x2="63.119" y2="571.627" width="0.6096" layer="21" curve="-42.907665"/>
+<wire x1="63.119" y1="571.627" x2="63.119" y2="98.425" width="0.6096" layer="21"/>
+<wire x1="63.119" y1="98.425" x2="62.23" y2="96.52" width="0.6096" layer="21"/>
+<wire x1="62.23" y1="96.52" x2="34.29" y2="64.008" width="0.6096" layer="21"/>
 <wire x1="34.29" y1="64.008" x2="44.069" y2="51.308" width="0.6096" layer="21" curve="118.93816"/>
 <wire x1="44.069" y1="51.308" x2="59.182" y2="51.181" width="0.6096" layer="21"/>
@@
 <wire x1="58.928" y1="37.338" x2="21.844" y2="37.465" width="0.6096" layer="21"/>
 <wire x1="21.844" y1="37.465" x2="15.113" y2="45.212" width="0.6096" layer="21" curve="-101.889589"/>
-<wire x1="15.113" y1="45.212" x2="31.242" y2="559.054" width="0.6096" layer="21"/>
+<wire x1="15.113" y1="45.212" x2="49.276" y2="571.881" width="0.6096" layer="21"/>
 <wire x1="76.2" y1="-50.8" x2="76.2" y2="723.9" width="0.254" layer="49" style="longdash"/>
+<dimension x1="51.308" y1="562.991" x2="63.184034375" y2="547.856940625" x3="67.999275" y3="541.7207" textsize="5.08" textratio="15" layer="47" dtype="radius" unit="inch"/>
+<wire x1="63.754" y1="540.766" x2="63.754" y2="566.166" width="2.3622" layer="108" style="shortdash"/>
+<wire x1="63.119" y1="566.293" x2="63.119" y2="540.893" width="1.0922" layer="108"/>
+<wire x1="89.916" y1="566.166" x2="89.916" y2="540.766" width="2.3622" layer="108" style="shortdash"/>
+<wire x1="90.551" y1="540.639" x2="90.551" y2="566.039" width="1.0922" layer="108"/>
 </plain>
 <attributes>
@@
 </autorouter>
 <elements>
-<element name="E$1" library="uarm_alignment_base" package="CARTRIDGE_ESP32" value="" x="25.4" y="673.1" rot="R270"/>
+<element name="E$1" library="uarm_alignment_base" package="CARTRIDGE_ESP32" value="" x="20.955" y="582.676" rot="R270"/>
 <element name="E$2" library="SparkFun-Hardware" package="ACTOBOTICS_CHANNEL_SINGLE_DRILL_REF" value="" x="0" y="571.5"/>
 <element name="E$3" library="SparkFun-Hardware" package="ACTOBOTICS_CHANNEL_SINGLE_DRILL_REF" value="" x="114.3" y="571.5"/>
 <element name="E$4" library="SparkFun-Hardware" package="ACTOBOTICS_CHANNEL_SINGLE_DRILL_REF" value="" x="0" y="0"/>
 <element name="E$5" library="SparkFun-Hardware" package="ACTOBOTICS_CHANNEL_SINGLE_DRILL_REF" value="" x="114.3" y="0"/>
-<element name="E$6" library="uarm_alignment_base" package="TUBE_&amp;_BEARING_1/2&quot;" value="" x="38.1" y="558.8"/>
+<element name="E$6" library="uarm_alignment_base" package="TUBE_&amp;_BEARING_1/2&quot;" value="" x="56.134" y="571.627"/>
 <element name="E$7" library="uarm_alignment_base" package="GEAR_84T" value="" x="109.601" y="60.325"/>
 <element name="E$8" library="uarm_alignment_base" package="GEAR_84T" value="" x="42.799" y="60.325"/>
 <element name="E$9" library="uarm_alignment_base" package="TUBE_&amp;_BEARING_1/2&quot;" value="" x="58.547" y="44.196"/>
 <element name="E$10" library="uarm_alignment_base" package="TUBE_&amp;_BEARING_1/2&quot;" value="" x="21.844" y="44.069"/>
-<element name="E$11" library="SparkFun-Hardware" package="ACTOBOTICS_CHANNEL_SINGLE_DRILL_REF" value="" x="0" y="508"/>
-<element name="E$12" library="SparkFun-Hardware" package="ACTOBOTICS_CHANNEL_SINGLE_DRILL_REF" value="" x="114.3" y="508"/>
+<element name="E$11" library="SparkFun-Hardware" package="ACTOBOTICS_CHANNEL_SINGLE_DRILL_REF" value="" x="0" y="533.4"/>
+<element name="E$12" library="SparkFun-Hardware" package="ACTOBOTICS_CHANNEL_SINGLE_DRILL_REF" value="" x="114.3" y="533.4"/>
 </elements>
 <signals>

Commit message: more belt fine tuning
added servo package

added 1/4" cutouts for inner wall sides to "punch" in
Parts:
- added E$13: (no value), uarm_alignment_base:SERVO_WITH_16T_GEAR_REF
- added E$14, E$15, E$16, E$17, E$18, E$19, E$20, E$21, E$22, E$23, E$24, E$25, E$26, E$27, E$28, E$29, E$30, E$31: (no value), uarm_alignment_base:1/4"_RECT_CUT_OUT
- moved E$8 0.05 mm to (42.8, 60.3)
- moved E$7 0.05 mm to (109.6, 60.3)
Other:
- board outline added: 21.6 x 51.7 mm
Changed lines of the file:
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@@
 <setting verticaltext="up"/>
 </settings>
-<grid distance="0.5" unitdist="inch" unit="inch" style="lines" multiple="1" display="yes" altdistance="0.05" altunitdist="inch" altunit="inch"/>
+<grid distance="0.5" unitdist="inch" unit="inch" style="lines" multiple="1" display="yes" altdistance="0.005" altunitdist="inch" altunit="inch"/>
 <layers>
 <layer number="1" name="Top" color="4" fill="1" visible="yes" active="yes"/>
@@
 <layer number="45" name="Holes" color="7" fill="1" visible="yes" active="yes"/>
 <layer number="46" name="Milling" color="3" fill="1" visible="no" active="yes"/>
-<layer number="47" name="Measures" color="7" fill="1" visible="yes" active="yes"/>
+<layer number="47" name="Measures" color="7" fill="1" visible="no" active="yes"/>
 <layer number="48" name="Document" color="7" fill="1" visible="no" active="yes"/>
 <layer number="49" name="Reference" color="13" fill="1" visible="yes" active="yes"/>
@@
 <layer number="106" name="bPlate" color="7" fill="1" visible="no" active="yes"/>
 <layer number="107" name="Crop" color="7" fill="1" visible="no" active="yes"/>
-<layer number="108" name="tplace-old" color="10" fill="1" visible="yes" active="yes"/>
+<layer number="108" name="tplace-old" color="10" fill="1" visible="no" active="yes"/>
 <layer number="109" name="ref-old" color="11" fill="1" visible="no" active="yes"/>
 <layer number="110" name="fp0" color="7" fill="1" visible="no" active="yes"/>
@@
 <wire x1="59.309" y1="571.5" x2="59.309" y2="99.06" width="6.35" layer="51"/>
 <wire x1="94.361" y1="571.5" x2="94.361" y2="99.06" width="6.35" layer="51"/>
-<circle x="48.910396875" y="19.00886875" radius="7.184203125" width="0.254" layer="49"/>
-<wire x1="78.013765625" y1="23.162221875" x2="74.970409375" y2="5.90248125" width="0.254" layer="49"/>
 <wire x1="74.970409375" y1="5.90248125" x2="74.676159375" y2="5.696446875" width="0.254" layer="49" curve="-90"/>
-<wire x1="74.676159375" y1="5.696446875" x2="37.405125" y2="12.268334375" width="0.254" layer="49"/>
-<wire x1="37.405125" y1="12.268334375" x2="40.448484375" y2="29.528075" width="0.254" layer="49"/>
-<wire x1="40.448484375" y1="29.528075" x2="40.74273125" y2="29.7341125" width="0.254" layer="49" curve="-90"/>
-<wire x1="40.74273125" y1="29.7341125" x2="78.013765625" y2="23.162221875" width="0.254" layer="49"/>
 <text x="36.83" y="72.39" size="1.778" layer="49" font="vector" ratio="15">84T</text>
 <wire x1="49.276" y1="571.881" x2="55.372" y2="578.358" width="0.6096" layer="21" curve="-83.121022"/>
@@
 <element name="E$5" library="SparkFun-Hardware" package="ACTOBOTICS_CHANNEL_SINGLE_DRILL_REF" value="" x="114.3" y="0"/>
 <element name="E$6" library="uarm_alignment_base" package="TUBE_&amp;_BEARING_1/2&quot;" value="" x="56.134" y="571.627"/>
-<element name="E$7" library="uarm_alignment_base" package="GEAR_84T" value="" x="109.601" y="60.325"/>
-<element name="E$8" library="uarm_alignment_base" package="GEAR_84T" value="" x="42.799" y="60.325"/>
+<element name="E$7" library="uarm_alignment_base" package="GEAR_84T" value="" x="109.5502" y="60.325"/>
+<element name="E$8" library="uarm_alignment_base" package="GEAR_84T" value="" x="42.8498" y="60.325"/>
 <element name="E$9" library="uarm_alignment_base" package="TUBE_&amp;_BEARING_1/2&quot;" value="" x="58.547" y="44.196"/>
 <element name="E$10" library="uarm_alignment_base" package="TUBE_&amp;_BEARING_1/2&quot;" value="" x="21.844" y="44.069"/>
 <element name="E$11" library="SparkFun-Hardware" package="ACTOBOTICS_CHANNEL_SINGLE_DRILL_REF" value="" x="0" y="533.4"/>
 <element name="E$12" library="SparkFun-Hardware" package="ACTOBOTICS_CHANNEL_SINGLE_DRILL_REF" value="" x="114.3" y="533.4"/>
+<element name="E$13" library="uarm_alignment_base" package="SERVO_WITH_16T_GEAR_REF" value="" x="30.4644375" y="98.162190625" rot="R90"/>
+<element name="E$14" library="uarm_alignment_base" package="1/4&quot;_RECT_CUT_OUT" value="" x="59.309" y="127"/>
+<element name="E$15" library="uarm_alignment_base" package="1/4&quot;_RECT_CUT_OUT" value="" x="59.309" y="177.8"/>
+<element name="E$16" library="uarm_alignment_base" package="1/4&quot;_RECT_CUT_OUT" value="" x="59.309" y="228.6"/>
+<element name="E$17" library="uarm_alignment_base" package="1/4&quot;_RECT_CUT_OUT" value="" x="59.309" y="279.4"/>
+<element name="E$18" library="uarm_alignment_base" package="1/4&quot;_RECT_CUT_OUT" value="" x="59.309" y="330.2"/>
+<element name="E$19" library="uarm_alignment_base" package="1/4&quot;_RECT_CUT_OUT" value="" x="59.309" y="381"/>
+<element name="E$20" library="uarm_alignment_base" package="1/4&quot;_RECT_CUT_OUT" value="" x="59.309" y="431.8"/>
+<element name="E$21" library="uarm_alignment_base" package="1/4&quot;_RECT_CUT_OUT" value="" x="59.309" y="482.6"/>
+<element name="E$22" library="uarm_alignment_base" package="1/4&quot;_RECT_CUT_OUT" value="" x="59.309" y="533.4"/>
+<element name="E$23" library="uarm_alignment_base" package="1/4&quot;_RECT_CUT_OUT" value="" x="94.361" y="127"/>
+<element name="E$24" library="uarm_alignment_base" package="1/4&quot;_RECT_CUT_OUT" value="" x="94.361" y="177.8"/>
+<element name="E$25" library="uarm_alignment_base" package="1/4&quot;_RECT_CUT_OUT" value="" x="94.361" y="228.6"/>
+<element name="E$26" library="uarm_alignment_base" package="1/4&quot;_RECT_CUT_OUT" value="" x="94.361" y="279.4"/>
+<element name="E$27" library="uarm_alignment_base" package="1/4&quot;_RECT_CUT_OUT" value="" x="94.361" y="330.2"/>
+<element name="E$28" library="uarm_alignment_base" package="1/4&quot;_RECT_CUT_OUT" value="" x="94.361" y="381"/>
+<element name="E$29" library="uarm_alignment_base" package="1/4&quot;_RECT_CUT_OUT" value="" x="94.361" y="431.8"/>
+<element name="E$30" library="uarm_alignment_base" package="1/4&quot;_RECT_CUT_OUT" value="" x="94.361" y="482.6"/>
+<element name="E$31" library="uarm_alignment_base" package="1/4&quot;_RECT_CUT_OUT" value="" x="94.361" y="533.4"/>
 </elements>
 <signals>
