File: Hardware_design/Cartridge_belt.brd (EAGLE design)
At the start: 21.6 x 51.7 mm, 31 parts

Commit message: A ot more work on belt drive system
Parts arrived, so used calipers to better fine tune all packages.

Building out library to include some END CAP parts, and mating drills
into other packages.

Has to slightly modify the position of some of the free pullies. I did
my best to not adjust the belt length, but this could result in needed
some more fine tuning to get the tension perfect later.
Parts:
- added E$32: (no value), uarm_alignment_base:END_STOP_CAP_1/2"_TUBE
- added E$33: (no value), uarm_alignment_base:END_STOP_CAP_1/4"_ROD
- E$11, E$12, E$4, E$5: device SparkFun-Hardware:ACTOBOTICS_CHANNEL_SINGLE_DRILL_REF -> uarm_alignment_base:ACTOBOTICS_1/2_HOLE_WITH_HUB_HOLES
- moved E$5 585.1 mm to (-59.1, 558.8), flipped to the bottom, turned to 270 degrees
- moved E$4 561.9 mm to (59.1, 558.8), turned to 270 degrees
- moved E$11 519.6 mm to (-59.1, 17.1), flipped to the bottom, turned to 180 degrees
- moved E$12 519.2 mm to (59.1, 17.1), turned to 180 degrees
- moved E$1 137.1 mm to (-95.3, 655.3), turned to 180 degrees
- moved E$9 76.2 mm to (-17.7, 42.9), turned to 45 degrees
- moved E$10 76.2 mm to (-54.4, 44.7), turned to 135 degrees
- moved E$2 76.2 mm to (-76.2, 571.5)
- moved E$23 76.2 mm to (18.2, 127.0)
- moved E$24 76.2 mm to (18.2, 177.8)
- moved E$25 76.2 mm to (18.2, 228.6)
- moved E$26 76.2 mm to (18.2, 279.4)
- moved E$27 76.2 mm to (18.2, 330.2)
- moved E$28 76.2 mm to (18.2, 381.0)
- moved E$29 76.2 mm to (18.2, 431.8)
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Other:
- board text removed: "84T"
