File: Hardware_design/Cartridge_belt.brd (EAGLE design)
At the start: 21.6 x 53.5 mm, 33 parts

Commit message: belt drive work
added hinges for WF

created inner wall that mates with teeth cuttouts

created hinge spacer in library as package. added 4 to unused space on
belt drive wall.
Parts:
- added E$34, E$35, E$36, E$37: (no value), Testing:HINGE_PM
- added E$38, E$39: (no value), uarm_alignment_base:ACTOBOTICS_1/2_HOLE_WITH_HUB_HOLES
- added E$40, E$41, E$42, E$43: (no value), uarm_alignment_base:HINGE_SPACER
- added E$44, E$49, E$50, E$51, E$52, E$53, E$54, E$55, E$56, E$57, E$58, E$59, E$60, E$61, E$62, E$63, E$64, E$65, E$66: (no value), uarm_alignment_base:1/4"_RECT_CUT_OUT
- added E$45, E$47, E$48: (no value), uarm_alignment_base:TUBE_&_BEARING_1/2"
- added E$46: (no value), uarm_alignment_base:GEAR_84T
- E$7: device uarm_alignment_base:GEAR_84T -> uarm_alignment_base:1/4"_RECT_CUT_OUT
- moved E$1 322.0 mm to (202.0, 531.6), turned to 270 degrees
- moved E$7 109.1 mm to (91.8, 152.4)
- moved E$23 1.27 mm to (16.9, 127.0)
- moved E$24 1.27 mm to (16.9, 177.8)
- moved E$25 1.27 mm to (16.9, 228.6)
- moved E$26 1.27 mm to (16.9, 279.4)
- moved E$27 1.27 mm to (16.9, 330.2)
- moved E$28 1.27 mm to (16.9, 381.0)
- moved E$29 1.27 mm to (16.9, 431.8)
- moved E$30 1.27 mm to (16.9, 482.6)
- moved E$31 1.27 mm to (16.9, 533.4)
Other:
- board size 21.6 x 53.5 mm -> 99 x 475 mm

Commit message: adjusted teeth sizes updated dxf
Note these teeth sizes worked at 9% speed, 100% power, 5K freq, in one
single pass.
The male teeth are 0.25" by 1".

The female teeth cutouts are 0.235" by 0.993"
Parts:
- E$14, E$15, E$16, E$17, E$18, E$19, E$20, E$21, E$22, E$23, E$24, E$25, E$26, E$27, E$28, E$29, E$30, E$31: device uarm_alignment_base:1/4"_RECT_CUT_OUT -> uarm_alignment_base:1/4_RECT_CUT_OUT_REDUCED_0.993_X_0.225
- E$44, E$49, E$50, E$51, E$52, E$53, E$54, E$55, E$56, E$57, E$58, E$59, E$61, E$62, E$63, E$64, E$65, E$66, E$7: device uarm_alignment_base:1/4"_RECT_CUT_OUT -> uarm_alignment_base:1/4"_RECT_CUT_OUT_1:1
Other:
- board size 99 x 475 mm -> 263.8 x 609.6 mm

Commit message: belt tension corrections
Brought down the entire top about 1/2". The original design was too
tight for the belt to even get in there. With the bearing removed
(effectively bringing the top roller down 1/2" inch), it was able to be
placed loosely.

Added tentioning slots, where I can place a 1/2" rod with clamps and add
tension to the belt.

designed the inner wall.

Removed hinges, I don't plan on having an opening or waffle top on this.
I'd like the tech to load from top (just like the uarm will do). They
can manually move the belt one board space by pressing the "up" or
"down" buttons.
Parts:
- removed E$40, E$41, E$42, E$43: (no value), uarm_alignment_base:HINGE_SPACER
- added E$100, E$72, E$82, E$83, E$84, E$85, E$86, E$87, E$88, E$89, E$90, E$91, E$92, E$93, E$94, E$95, E$96, E$97, E$98, E$99: (no value), uarm_alignment_base:1/4"_RECT_CUT_OUT_1:1
- added E$67, E$68, E$69, E$70, E$71: (no value), uarm_alignment_base:1/4_RECT_CUT_OUT_REDUCED_0.993_X_0.225
- E$34, E$35, E$36, E$37: device Testing:HINGE_PM -> uarm_alignment_base:1/4_RECT_CUT_OUT_REDUCED_0.993_X_0.225
- E$60: device uarm_alignment_base:1/4"_RECT_CUT_OUT -> uarm_alignment_base:1/4"_RECT_CUT_OUT_1:1
- moved E$34 411.9 mm to (117.9, 127.0), turned to 0 degrees
- moved E$37 143.7 mm to (117.9, 279.4), turned to 0 degrees
- moved E$1 106.8 mm to (196.5, 638.2)
- moved E$36 84.2 mm to (117.9, 228.6), turned to 0 degrees
- moved E$35 71.8 mm to (117.9, 177.8), turned to 0 degrees
- moved E$2 6.35 mm to (-76.2, 565.1)
- moved E$3 6.35 mm to (38.1, 565.1)
- moved E$38 6.35 mm to (-57.1, 584.2)
- moved E$39 6.35 mm to (57.1, 584.2)
- moved E$4 6.35 mm to (59.1, 552.5)
- moved E$45 6.35 mm to (20.1, 565.3)
- moved E$5 6.35 mm to (-59.1, 552.5)
- moved E$6 6.35 mm to (-20.1, 565.3)
Other:
- board size 263.8 x 609.6 mm -> 350.2 x 603.2 mm

Commit message: adjusted for correct width of inner slot
Parts:
- moved E$1 148.6 mm to (56.8, 689.0)
- moved E$100 1.30 mm to (272.2, 101.6)
- moved E$91 1.30 mm to (272.2, 152.4)
- moved E$92 1.30 mm to (272.2, 203.2)
- moved E$93 1.30 mm to (272.2, 254.0)
- moved E$94 1.30 mm to (272.2, 304.8)
- moved E$95 1.30 mm to (272.2, 355.6)
- moved E$96 1.30 mm to (272.2, 406.4)
- moved E$97 1.30 mm to (272.2, 457.2)
- moved E$98 1.30 mm to (272.2, 508.0)
- moved E$99 1.30 mm to (272.2, 558.8)
- moved E$45 0.72 mm to (20.8, 565.2)
- moved E$6 0.72 mm to (-20.8, 565.2)
- moved E$14 0.64 mm to (-17.5, 127.0)
- moved E$15 0.64 mm to (-17.5, 177.8)
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Other:
- board size 350.2 x 603.2 mm -> 351.5 x 603.2 mm
